File: Power.kicad_sch (KiCad schematic)
At the start: 33 parts, among them J1 Barrel_Jack_MountingPin, J2 USB_B_Micro, U1 LM2596S-5, U3 LM1117-3.3, U4 LM1117-1.8, U5 TPS2552DBVR

Commit message: Schematic updated
Parts:
- added J9: VBus-Select, Connector_PinHeader_2.54mm:PinHeader_1x03_P2.54mm_Vertical, symbol Connector_Generic:Conn_01x03
- R5: value 20k -> 47k
Connections:
- net +5V: now also R6.1
- net VBUS: no longer R6.1
Other:
- note added: "USB OVERCURRENT"
- note removed: "USB OVERCURRENT/NOT COMPLETED"
- moved on the sheet: R5, R6
Changed lines of the file:
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@@
     (stroke (width 0) (type default) (color 0 0 0 0))
   )
-  (wire (pts (xy 132.842 163.322) (xy 132.842 169.672))
+  (wire (pts (xy 137.414 154.432) (xy 137.414 160.782))
     (stroke (width 0) (type default) (color 0 0 0 0))
   )
@@
     (stroke (width 0) (type default) (color 0 0 0 0))
   )
-  (wire (pts (xy 132.842 155.702) (xy 132.842 158.242))
+  (wire (pts (xy 137.414 146.812) (xy 137.414 149.352))
     (stroke (width 0) (type default) (color 0 0 0 0))
   )
@@
     (stroke (width 0) (type default) (color 0 0 0 0))
   )
-  (wire (pts (xy 116.84 162.56) (xy 116.84 167.132))
+  (wire (pts (xy 121.412 153.67) (xy 121.412 158.242))
     (stroke (width 0) (type default) (color 0 0 0 0))
   )
@@
     (stroke (width 0) (type default) (color 0 0 0 0))
   )
-  (wire (pts (xy 116.84 153.162) (xy 116.84 157.48))
+  (wire (pts (xy 121.412 144.272) (xy 121.412 148.59))
     (stroke (width 0) (type default) (color 0 0 0 0))
   )
@@
     (effects (font (size 2.5 2.5) (thickness 0.5) bold) (justify left bottom))
   )
-  (text "USB OVERCURRENT/NOT COMPLETED" (at 22.86 137.795 0)
+  (text "USB OVERCURRENT" (at 22.86 137.795 0)
     (effects (font (size 2.5 2.5) (thickness 0.5) bold) (justify left bottom))
   )
@@
     (effects (font (size 2.5 2.5) (thickness 0.5) bold) (justify left bottom))
   )
-  (label "USB_ILIM" (at 116.84 153.162 0)
+  (label "USB_ILIM" (at 121.412 144.272 0)
     (effects (font (size 1.27 1.27)) (justify left bottom))
   )
@@
     (effects (font (size 1.27 1.27)) (justify left bottom))
   )
-  (label "USB_FAULT" (at 132.842 169.672 0)
+  (label "USB_FAULT" (at 137.414 160.782 0)
     (effects (font (size 1.27 1.27)) (justify left bottom))
   )
@@
     (pin "2")
   )
+  (symbol (lib_id "Connector_Generic:Conn_01x03") (at 131.064 177.292 270) (unit 1)
+    (in_bom yes) (on_board yes) (fields_autoplaced)
+    (property "Reference" "J9" (id 0) (at 135.636 176.0219 90)
+      (effects (font (size 1.27 1.27)) (justify left))
+    )
+    (property "Value" "VBus-Select" (id 1) (at 135.636 178.5619 90)
+      (effects (font (size 1.27 1.27)) (justify left))
+    )
+    (property "Footprint" "Connector_PinHeader_2.54mm:PinHeader_1x03_P2.54mm_Vertical" (id 2) (at 131.064 177.292 0)
+      (effects (font (size 1.27 1.27)) hide)
+    )
+    (property "Datasheet" "~" (id 3) (at 131.064 177.292 0)
+      (effects (font (size 1.27 1.27)) hide)
+    )
+    (pin "1")
+    (pin "2")
+    (pin "3")
+  )
   (symbol (lib_id "Device:R_Small_US") (at 256.54 125.73 90) (unit 1)
     (in_bom yes) (on_board yes)
@@
     (pin "1")
   )
-  (symbol (lib_id "Device:R_Small_US") (at 116.84 160.02 0) (unit 1)
-    (in_bom yes) (on_board yes)
-    (property "Reference" "R5" (id 0) (at 118.11 158.75 0)
-      (effects (font (size 1.27 1.27)) (justify left))
-    )
-    (property "Value" "20k" (id 1) (at 118.11 161.29 0)
-      (effects (font (size 1.27 1.27)) (justify left))
-    )
-    (property "Footprint" "Resistor_SMD:R_0603_1608Metric" (id 2) (at 116.84 160.02 0)
-      (effects (font (size 1.27 1.27)) hide)
-    )
-    (property "Datasheet" "~" (id 3) (at 116.84 160.02 0)
+  (symbol (lib_id "Device:R_Small_US") (at 121.412 151.13 0) (unit 1)
+    (in_bom yes) (on_board yes)
+    (property "Reference" "R5" (id 0) (at 122.682 149.86 0)
+      (effects (font (size 1.27 1.27)) (justify left))
+    )
+    (property "Value" "47k" (id 1) (at 122.682 152.4 0)
+      (effects (font (size 1.27 1.27)) (justify left))
+    )
+    (property "Footprint" "Resistor_SMD:R_0603_1608Metric" (id 2) (at 121.412 151.13 0)
+      (effects (font (size 1.27 1.27)) hide)
+    )
+    (property "Datasheet" "~" (id 3) (at 121.412 151.13 0)
       (effects (font (size 1.27 1.27)) hide)
     )
@@
     (pin "1")
   )
+  (symbol (lib_id "power:+5V") (at 137.414 146.812 0) (unit 1)
+    (in_bom yes) (on_board yes)
+    (property "Reference" "#PWR0111" (id 0) (at 137.414 150.622 0)
+      (effects (font (size 1.27 1.27)) hide)
+    )
+    (property "Value" "+5V" (id 1) (at 137.16 143.002 0))
+    (property "Footprint" "" (id 2) (at 137.414 146.812 0)
+      (effects (font (size 1.27 1.27)) hide)
+    )
+    (property "Datasheet" "" (id 3) (at 137.414 146.812 0)
+      (effects (font (size 1.27 1.27)) hide)
+    )
+    (pin "1")
+  )
   (symbol (lib_id "Regulator_Switching:LM2596S-5") (at 55.88 38.1 0) (unit 1)
     (in_bom yes) (on_board yes) (fields_autoplaced)
@@
     (pin "1")
   )
-  (symbol (lib_id "power:GND") (at 116.84 167.132 0) (unit 1)
-    (in_bom yes) (on_board yes) (fields_autoplaced)
-    (property "Reference" "#PWR0127" (id 0) (at 116.84 173.482 0)
-      (effects (font (size 1.27 1.27)) hide)
-    )
-    (property "Value" "GND" (id 1) (at 116.84 172.212 0))
-    (property "Footprint" "" (id 2) (at 116.84 167.132 0)
-      (effects (font (size 1.27 1.27)) hide)
-    )
-    (property "Datasheet" "" (id 3) (at 116.84 167.132 0)
+  (symbol (lib_id "power:GND") (at 121.412 158.242 0) (unit 1)
+    (in_bom yes) (on_board yes) (fields_autoplaced)
+    (property "Reference" "#PWR0127" (id 0) (at 121.412 164.592 0)
+      (effects (font (size 1.27 1.27)) hide)
+    )
+    (property "Value" "GND" (id 1) (at 121.412 163.322 0))
+    (property "Footprint" "" (id 2) (at 121.412 158.242 0)
+      (effects (font (size 1.27 1.27)) hide)
+    )
+    (property "Datasheet" "" (id 3) (at 121.412 158.242 0)
       (effects (font (size 1.27 1.27)) hide)
     )
@@
     (pin "1")
   )
-  (symbol (lib_id "Device:R_Small_US") (at 132.842 160.782 0) (unit 1)
-    (in_bom yes) (on_board yes)
-    (property "Reference" "R6" (id 0) (at 134.112 159.512 0)
-      (effects (font (size 1.27 1.27)) (justify left))
-    )
-    (property "Value" "100k" (id 1) (at 134.112 162.052 0)
-      (effects (font (size 1.27 1.27)) (justify left))
-    )
-    (property "Footprint" "Resistor_SMD:R_0603_1608Metric" (id 2) (at 132.842 160.782 0)
-      (effects (font (size 1.27 1.27)) hide)
-    )
-    (property "Datasheet" "~" (id 3) (at 132.842 160.782 0)
+  (symbol (lib_id "Device:R_Small_US") (at 137.414 151.892 0) (unit 1)
+    (in_bom yes) (on_board yes)
+    (property "Reference" "R6" (id 0) (at 138.684 150.622 0)
+      (effects (font (size 1.27 1.27)) (justify left))
+    )
+    (property "Value" "100k" (id 1) (at 138.684 153.162 0)
+      (effects (font (size 1.27 1.27)) (justify left))
+    )
+    (property "Footprint" "Resistor_SMD:R_0603_1608Metric" (id 2) (at 137.414 151.892 0)
+      (effects (font (size 1.27 1.27)) hide)
+    )
+    (property "Datasheet" "~" (id 3) (at 137.414 151.892 0)
       (effects (font (size 1.27 1.27)) hide)
     )
@@
     (pin "2")
   )
-  (symbol (lib_id "power:VBUS") (at 132.842 155.702 0) (unit 1)
-    (in_bom yes) (on_board yes)
-    (property "Reference" "#PWR0111" (id 0) (at 132.842 159.512 0)
-      (effects (font (size 1.27 1.27)) hide)
-    )
-    (property "Value" "VBUS" (id 1) (at 135.382 151.892 0)
-      (effects (font (size 1.27 1.27)) (justify right))
-    )
-    (property "Footprint" "" (id 2) (at 132.842 155.702 0)
-      (effects (font (size 1.27 1.27)) hide)
-    )
-    (property "Datasheet" "" (id 3) (at 132.842 155.702 0)
-      (effects (font (size 1.27 1.27)) hide)
-    )
-    (pin "1")
-  )
   (symbol (lib_id "Connector:Barrel_Jack_MountingPin") (at 172.974 37.592 0) (unit 1)
     (in_bom yes) (on_board yes) (fields_autoplaced)
@@
   )
   (symbol (lib_id "power:+5V") (at 28.448 154.686 0) (unit 1)
-    (in_bom yes) (on_board yes) (fields_autoplaced)
+    (in_bom yes) (on_board yes)
     (property "Reference" "#PWR0112" (id 0) (at 28.448 158.496 0)
       (effects (font (size 1.27 1.27)) hide)
     )
-    (property "Value" "+5V" (id 1) (at 28.448 148.971 0))
+    (property "Value" "+5V" (id 1) (at 28.194 150.876 0))
     (property "Footprint" "" (id 2) (at 28.448 154.686 0)
       (effects (font (size 1.27 1.27)) hide)

Commit message: JTAG swo pin pull down yapıldı
Parts:
- C17, C19: value 10uF -> 100uF
Connections:
- net VBUS: now also J9.2 (Pin_2)
- no-connect marks 4 -> 3
Changed lines of the file:
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@@
   (junction (at 61.595 89.535) (diameter 0) (color 0 0 0 0)
   )
-  (no_connect (at 159.004 43.688))
   (no_connect (at 172.974 46.482))
   (no_connect (at 156.21 41.91))
@@
     (pin "1")
   )
+  (symbol (lib_id "power:VBUS") (at 131.064 172.212 0) (mirror y) (unit 1)
+    (in_bom yes) (on_board yes)
+    (property "Reference" "#PWR0145" (id 0) (at 131.064 176.022 0)
+      (effects (font (size 1.27 1.27)) hide)
+    )
+    (property "Value" "VBUS" (id 1) (at 128.524 168.402 0)
+      (effects (font (size 1.27 1.27)) (justify right))
+    )
+    (property "Footprint" "" (id 2) (at 131.064 172.212 0)
+      (effects (font (size 1.27 1.27)) hide)
+    )
+    (property "Datasheet" "" (id 3) (at 131.064 172.212 0)
+      (effects (font (size 1.27 1.27)) hide)
+    )
+    (pin "1")
+  )
   (symbol (lib_id "Device:C_Polarized") (at 116.84 99.695 0) (unit 1)
     (in_bom yes) (on_board yes)
@@
       (effects (font (size 1.27 1.27)) (justify left))
     )
-    (property "Value" "10uF" (id 1) (at 119.38 100.33 0)
+    (property "Value" "100uF" (id 1) (at 119.38 100.33 0)
       (effects (font (size 1.27 1.27)) (justify left))
     )
@@
       (effects (font (size 1.27 1.27)) (justify left))
     )
-    (property "Value" "10uF" (id 1) (at 64.135 100.33 0)
-      (effects (font (size 1.27 1.27)) (justify left))
-    )
+    (property "Value" "100uF" (id 1) (at 64.135 100.33 0)
+      (effects (font (size 1.27 1.27)) (justify left))
+    )

Commit message: Butonlar eklendi
Parts:
- J3: renamed from J1; value Barrel_Jack_MountingPin -> DC_IN
- renumbered C4 to C3, C17 to C4, C18 to C5, C20 to C6, C3 to C7, C5 to C8, C19 to C9, J9 to J1, R5 to R1, R6 to R2, R1 to R3, R2 to R4, R3 to R5, R4 to R6, TP6 to TP1, TP5 to TP2, TP1 to TP3, TP2 to TP4, TP4 to TP5, TP3 to TP6, U5 to U1, U3 to U2, U1 to U3

Commit message: Butonlar eklendi ve usb eklendi
Connections:
- net USB0_VBUS: now reaches J1.1 (Pin_1)
- net USB0_VBUS: now also J1.3 (Pin_3)
Changed lines of the file:
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@@
+    (stroke (width 0) (type default) (color 0 0 0 0))
+  )
+  (wire (pts (xy 133.604 168.91) (xy 139.446 168.91))
     (stroke (width 0) (type default) (color 0 0 0 0))
   )
@@
     (stroke (width 0.5) (type solid) (color 57 87 255 1))
   )
+  (wire (pts (xy 128.524 168.656) (xy 128.524 172.212))
+    (stroke (width 0) (type default) (color 0 0 0 0))
+  )
   (wire (pts (xy 116.84 89.535) (xy 116.84 95.885))
     (stroke (width 0) (type default) (color 0 0 0 0))
@@
     (stroke (width 0) (type default) (color 0 0 0 0))
   )
+  (wire (pts (xy 125.222 168.656) (xy 128.524 168.656))
+    (stroke (width 0) (type default) (color 0 0 0 0))
+  )
   (wire (pts (xy 148.59 52.07) (xy 148.59 56.515))
     (stroke (width 0) (type default) (color 0 0 0 0))
@@
   )
   (wire (pts (xy 73.025 40.64) (xy 82.55 40.64))
+    (stroke (width 0) (type default) (color 0 0 0 0))
+  )
+  (wire (pts (xy 133.604 172.212) (xy 133.604 168.91))
     (stroke (width 0) (type default) (color 0 0 0 0))
   )
@@
     (effects (font (size 1.27 1.27)) (justify left))
     (property "Intersheet References" "${INTERSHEET_REFS}" (id 0) (at 273.1045 37.3856 0)
+      (effects (font (size 1.27 1.27)) (justify left) hide)
+    )
+  )
+  (global_label "USB0_VBUS" (shape input) (at 139.446 168.91 0) (fields_autoplaced)
+    (effects (font (size 1.27 1.27)) (justify left))
+    (property "Intersheet References" "${INTERSHEET_REFS}" (id 0) (at 152.7448 168.9894 0)
       (effects (font (size 1.27 1.27)) (justify left) hide)
     )
@@
     )
   )
+  (global_label "USB0_VBUS" (shape input) (at 125.222 168.656 180) (fields_autoplaced)
+    (effects (font (size 1.27 1.27)) (justify right))
+    (property "Intersheet References" "${INTERSHEET_REFS}" (id 0) (at 111.9232 168.5766 0)
+      (effects (font (size 1.27 1.27)) (justify right) hide)
+    )
+  )
